File: PCB/termocuplaJ v2/termocuplaJ.sch (KiCad schematic (older format))
At the start: 42 parts, among them J1 Pad_NEWPIECE, J2 Pad_PIECE-RESET, J3 Conn_02x08_Odd_Even, J5 Conn_01x01_Female, K1 SANYOU_SRD_Form_C, K2 SANYOU_SRD_Form_C, Q1 PZT2222A, Q2 PZT2222A, U1 MCP601-xOT, U2 L7805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

Commit message: FINAL ENTREGADO
Other:
- note added: "Se ensamblo finalmente con el INA129 y R8=100K\ncon muy buenos resultados"
Changed lines of the file:
@@
 Text Notes 3400 4800 0    79   ~ 0
 Falta div.tension en \nSDI, SCK y CS\n2.2k a gnd es suf.\nSS le falta 1K en serie\npara completar el div.tension\n
+Text Notes 4450 5800 0    79   Italic 16
+Se ensamblo finalmente con el INA129 y R8=100K\ncon muy buenos resultados
 $EndSCHEMATC
